File: hardware/USupply/SYS_PW.kicad_sch (KiCad schematic)
At the start: 0 parts

Commit message: feat(hw/usb): update 3.3v circuit
Parts:
- added C2: 4.7uF, Capacitor_SMD:C_0603_1608Metric_Pad1.08x0.95mm_HandSolder, symbol Device:C
- added C2: 10uF, Capacitor_SMD:C_0603_1608Metric_Pad1.08x0.95mm_HandSolder, symbol Device:C
- added C2: 33pF, Capacitor_SMD:C_0603_1608Metric_Pad1.08x0.95mm_HandSolder, symbol Device:C
- added C2: 100nF, Capacitor_SMD:C_0603_1608Metric_Pad1.08x0.95mm_HandSolder, symbol Device:C
- added D5: D_Schottky, Diode_SMD:D_SOD-123, symbol Device:D_Schottky
- added L1: 4.7uH, Inductor_SMD:L_Taiyo-Yuden_MD-5050, symbol Device:L
- added R2: 200K, Resistor_SMD:R_0603_1608Metric, symbol Device:R
- added R2: 124K, Resistor_SMD:R_0603_1608Metric, symbol Device:R
- added R2: 100K, Resistor_SMD:R_0603_1608Metric, symbol Device:R
- added R2: 40.2K, Resistor_SMD:R_0603_1608Metric, symbol Device:R
- added U2: MP2451/MP2459, Package_TO_SOT_SMD:TSOT-23-6, symbol Regulator_Switching:MP2303ADN
Connections:
- new net: R2.1, R2.2, U2.4 (EN)
- new net: C2.1, R2.1, R2.1, U2.3 (FB)
- new net: C2.2, D5.1 (K), L1.1, U2.6 (SW)
- new net: C2.1, U2.1 (BST)
- new net 3V3: C2.1, C2.2, L1.2, R2.2
- new net GND: C2.2, C2.2, D5.2 (A), R2.2, R2.2, U2.2 (GND)
- new net VDC: C2.1, R2.1, U2.5 (VIN)
Other:
- note added: "(1%)"
- note added: "(X5R/X7R)"
